File: Carte_eagle/carte_realise/notre_carte.brd (EAGLE design)
At the start: 100 x 80 mm, 14 parts, among them CON1 CON-1X2-SPOX-M-2.50, CON2 CON-1X2-SPOX-M-2.50, U1 DOGM163

Commit message: mise a jour de la carte et board
Parts:
- removed R1_BOUT, R2_BOUT, R3_BOUT: 10k, rcl:0207/10
- moved C3 179.1 mm to (72.4, 66.0), turned to 180 degrees
- moved CON1 161.8 mm to (88.9, 44.5), turned to 90 degrees
- moved BOUTON_B 131.8 mm to (69.8, 10.2)
- moved CON2 124.5 mm to (88.9, 30.5), turned to 90 degrees
- moved U1 100.1 mm to (47.0, 36.8)
- moved C2 97.1 mm to (15.2, 16.5), turned to 180 degrees
- moved C1 94.6 mm to (15.2, 24.1), turned to 180 degrees
- moved BOUTON_N 86.8 mm to (48.3, 10.2)
- moved SV1 84.4 mm to (49.5, 66.0)
- moved BOUTON_R 78.5 mm to (26.7, 10.2)
- moved R_RETRO 52.1 mm to (15.2, 39.4), turned to 90 degrees
Connections:
- net +5V: now also BOUTON_B.3, BOUTON_N.3, BOUTON_R.3; no longer R1_BOUT.1, R2_BOUT.1, R3_BOUT.1
- net RE0_BOUT_B: no longer BOUTON_B.3, R1_BOUT.2
- net RE1_BOUT_N: no longer BOUTON_N.3, R2_BOUT.2
- net RE2_BOUT_R: no longer BOUTON_R.3, R3_BOUT.2
Routing:
- added copper zone on layer 1, net GND
